Commit message: Adding rear castor wheels and white color check for all channels

File: catkin_ws/src/my_robot/urdf/my_robot.xacro (robot description, xacro)
@@ -15,5 +15,5 @@
     <pose>0 0 0.1 0 0 0</pose>
     <inertial>
-      <mass value="15"/>
+      <mass value="15.0"/>
       <origin xyz="0 0 0" rpy="0 0 0"/>
       <inertia
@@ -23,4 +23,10 @@
       />
     </inertial>
+    <collision name='collision'>
+      <origin xyz="0 0 0" rpy=" 0 0 0"/>
+      <geometry>
+        <box size=".4 .2 .1"/>
+      </geometry>
+    </collision>
     <collision name="chassis_collision">
       <geometry>
@@ -32,4 +38,17 @@
       <geometry>
         <box size="0.5 0.25 0.07"/>
+      </geometry>
+    </visual>
+    <!--back caster-->
+    <collision name='back_caster_collision'>
+      <origin xyz="-0.15 0 -0.05" rpy=" 0 0 0"/>
+      <geometry>
+        <sphere radius="0.0499"/>
+      </geometry>
+    </collision>
+    <visual name='back_caster_visual'>
+      <origin xyz="-0.15 0 -0.05" rpy=" 0 0 0"/>
+      <geometry>
+        <sphere radius="0.05"/>
       </geometry>
     </visual>
